File: f13-tkl.kicad_pcb (KiCad board)
At the start: 2 copper layers, 202 parts, among them J1 Conn_01x04, Q1 2N7002, SW1 SW_Push, U1 MCP1700-3302E_SOT23, U2 STM32F072CBTx

Commit message: lots of changes
Parts:
- added D90: D_Schottky, Diode_SMD:D_SOD-123, B.Cu at (363.3, 128.8)
- added D91: D_TVS, Diode_SMD:D_SOD-123, B.Cu at (367.8, 119.1)
- added F1: 500mA, Fuse:Fuse_1206_3216Metric, B.Cu at (369.4, 113.8)
- added LOGO1: O-LOGO, board_logos:o-logo-300dpi, F.Cu at (250.8, 186.5)
- added LOGO2: O-LOGO, board_logos:o-logo-300dpi, B.Cu at (249.8, 186.5)
- added R5: 1k, Resistor_SMD:R_0603_1608Metric, B.Cu at (387.5, 96.3)
- MX16: value MX-NoLED -> MX-LED; footprint MX_Only:MXOnly-1U-NoLED -> MX_Only:MXOnly-1U
- moved R3 43.4 mm to (373.1, 163.7), turned to 270 degrees
- moved R1 42.8 mm to (366.1, 164.6), turned to 270 degrees
- moved R2 39.8 mm to (373.9, 166.1), turned to 180 degrees
- moved D32 39.3 mm to (354.3, 152.8)
- moved U1 34.8 mm to (366.8, 133.7), turned to 270 degrees
- moved C2 34.5 mm to (363.3, 133.5), turned to 270 degrees
- moved C1 33.1 mm to (367.2, 130.6), turned to 180 degrees
- moved C4 32.5 mm to (367.8, 164.6), turned to 90 degrees
- moved Q1 32.5 mm to (370.5, 163.8), turned to 180 degrees
- moved C3 30.7 mm to (374.8, 163.7), turned to 90 degrees
- moved D77 25.5 mm to (347.0, 171.8)
- moved J1 23.0 mm to (342.1, 100.8)
- moved D88 15.9 mm to (390.5, 190.9)
- moved C12 5.71 mm to (370.0, 158.8)
- moved C11 5.64 mm to (370.0, 157.2)
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Connections:
- J1 pad 1: +5V -> VCC
- MX54 pad 1: Col0 -> Net-(D53-Pad2)
- MX54 pad 2: Net-(D53-Pad2) -> Col0
- MX54 pad 3: GND -> +5V
- MX55 pad 3: GND -> +5V
- MX77 pad 2: Net-(MX77-Pad2) -> Net-(D75-Pad2)
- MX78 pad 2: Net-(MX78-Pad2) -> Net-(D76-Pad2)
- R4 pad 1: CAPS_LED -> CAPS
- U2 pad 12: Net-(U2-Pad12) -> Col13
- U2 pad 13: Net-(U2-Pad13) -> Row4
- U2 pad 14: Net-(U2-Pad14) -> Row5
- U2 pad 15: Net-(U2-Pad15) -> Row3
- U2 pad 16: Net-(U2-Pad16) -> Row0
- U2 pad 17: Net-(U2-Pad17) -> Col12
- U2 pad 18: Net-(U2-Pad18) -> Col11
- U2 pad 19: Net-(U2-Pad19) -> Col10
- U2 pad 20: Net-(U2-Pad20) -> Col9
- U2 pad 21: Net-(U2-Pad21) -> Col8
- U2 pad 22: Net-(U2-Pad22) -> Col7
- U2 pad 25: Net-(U2-Pad25) -> Col6
- U2 pad 26: Net-(U2-Pad26) -> Col5
- U2 pad 27: Net-(U2-Pad27) -> Col4
- U2 pad 28: Net-(U2-Pad28) -> Col3
- U2 pad 29: Net-(U2-Pad29) -> Col2
- U2 pad 30: Net-(U2-Pad30) -> Col1
- U2 pad 31: Net-(U2-Pad31) -> Col0
- U2 pad 38: Net-(U2-Pad38) -> SCROLL
- U2 pad 39: Net-(U2-Pad39) -> Row1
- U2 pad 40: Net-(U2-Pad40) -> Row2
- U2 pad 41: Net-(U2-Pad41) -> Col16
- U2 pad 42: Net-(U2-Pad42) -> Col15
- U2 pad 43: Net-(U2-Pad43) -> CAPS
- U2 pad 45: Net-(U2-Pad45) -> Col14
Routing:
- net Row0: track 0.00 -> 401.4 mm, vias 0 -> 2
- net Col0: track 0.00 -> 401.2 mm
- net +5V: track 0.00 -> 395.0 mm, vias 0 -> 4
- net +3V3: track 0.00 -> 393.0 mm, vias 0 -> 9
- net Col1: track 0.00 -> 381.0 mm
- net Row1: track 0.00 -> 371.8 mm, vias 0 -> 4
- net Row2: track 0.00 -> 365.0 mm, vias 0 -> 2
- net Col2: track 0.00 -> 358.9 mm
- net Row5: track 0.00 -> 354.4 mm, vias 0 -> 2
- net BOOT0: track 0.00 -> 333.9 mm, vias 0 -> 3
- net Row4: track 0.00 -> 321.1 mm, vias 0 -> 2
- net Col3: track 0.00 -> 316.0 mm
- net CAPS: track 0.00 -> 299.1 mm, vias 0 -> 2
- net Col4: track 0.00 -> 295.9 mm
- net Col6: track 0.00 -> 278.4 mm
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- added copper zone on B.Cu, net GND
Other:
- board outline added: 346.7 x 118.1 mm
- board text added: "+"
- board text added: "-"
- board text added: "7.00u"
