File: f13-tkl.sch (KiCad schematic (older format))
At the start: 20 parts

Commit message: finish schematic rev1
Parts:
- added D1, D10, D11, D12, D13, D14, D15, D16, D17, D18, D19, D2, D20, D21, D22, D23, D24, D25, D26, D27, D28, D29, D3, D30, D31, D32, D33, D34, D35, D36, D37, D38, D39, D4, D40, D41, D42, D43, D44, D45, D46, D47, D48, D49, D5, D50, D51, D52, D53, D54, D55, D56, D57, D58, D59, D6, D60, D61, D62, D63, D64, D65, D66, D67, D68, D69, D7, D70, D71, D72, D73, D74, D75, D76, D77, D78, D79, D8, D80, D81, D82, D83, D84, D85, D86, D87, D88, D89, D9: D_Small, Diode_SMD:D_SOD-123, symbol Device:D_Small
- added MX1, MX10, MX11, MX12, MX13, MX14, MX15, MX16, MX17, MX18, MX19, MX2, MX20, MX21, MX22, MX23, MX24, MX25, MX26, MX27, MX28, MX29, MX3, MX30, MX31, MX33, MX34, MX35, MX36, MX38, MX39, MX4, MX40, MX41, MX42, MX43, MX44, MX45, MX46, MX47, MX48, MX49, MX5, MX51, MX52, MX53, MX56, MX57, MX58, MX59, MX6, MX60, MX61, MX62, MX63, MX64, MX65, MX66, MX69, MX7, MX70, MX71, MX72, MX73, MX74, MX75, MX76, MX77, MX78, MX79, MX8, MX81, MX82, MX84, MX88, MX9, MX90, MX91, MX92: MX-NoLED, MX_Only:MXOnly-1U-NoLED, symbol MX_Alps_Hybrid:MX-NoLED
- added MX32: MX-NoLED, MX_Only:MXOnly-2U-NoLED, symbol MX_Alps_Hybrid:MX-NoLED
- added MX37, MX50, MX83, MX85, MX87, MX89: MX-NoLED, MX_Only:MXOnly-1.5U-NoLED, symbol MX_Alps_Hybrid:MX-NoLED
- added MX54: MX-LED, MX_Only:MXOnly-1.25U-FLIPPED, symbol MX_Alps_Hybrid:MX-LED
- added MX55: MX-LED, MX_Only:MXOnly-1.75U, symbol MX_Alps_Hybrid:MX-LED
- added MX67: MX-NoLED, MX_Only:MXOnly-2.25U-ReversedStabilizers-NoLED, symbol MX_Alps_Hybrid:MX-NoLED
- added MX68: MX-NoLED, MX_Only:MXOnly-2.25U-NoLED, symbol MX_Alps_Hybrid:MX-NoLED
- added MX80: MX-NoLED, MX_Only:MXOnly-2.75U-NoLED, symbol MX_Alps_Hybrid:MX-NoLED
- added MX86: MX-NoLED, MX_Only:MXOnly-7U-ReversedStabilizers-NoLED, symbol MX_Alps_Hybrid:MX-NoLED
- added R4: 1k, Resistor_SMD:R_0603_1608Metric, symbol Device:R_Small
- C1, C10, C11, C12, C2, C3, C4, C6, C7, C8, C9: renamed from C?; footprint (none) -> Capacitor_SMD:C_0603_1608Metric
- C5: renamed from C?; value 100nF -> 0.1uF; footprint (none) -> Capacitor_SMD:C_0603_1608Metric
- J1: renamed from J?; footprint (none) -> random-keyboard-parts:JST-SR-4
- R1, R2, R3: renamed from R?; footprint (none) -> Resistor_SMD:R_0603_1608Metric
- SW1: renamed from SW?; footprint (none) -> footprints-and-logos:K2-1187SQ-A4SW-06
- gave numbers to parts that had none: 3
Connections:
- net GND: now also MX54.4 (LEDGND), MX55.4 (LEDGND)
- new net: D1.2 (A), MX1.2 (ROW)
- new net: D14.2 (A), MX14.2 (ROW)
- new net: D15.2 (A), MX15.2 (ROW)
- new net: D16.2 (A), MX16.2 (ROW)
- new net: D17.2 (A), MX17.2 (ROW)
- new net: D87.2 (A), MX90.2 (ROW)
- new net: D88.2 (A), MX91.2 (ROW)
- new net: D89.2 (A), MX92.2 (ROW)
- new net: D79.2 (A), MX82.2 (ROW)
- new net: D18.2 (A), MX18.2 (ROW)
- new net: D19.2 (A), MX19.2 (ROW)
- new net: D20.2 (A), MX20.2 (ROW)
- new net: D21.2 (A), MX21.2 (ROW)
- new net: D22.2 (A), MX22.2 (ROW)
- new net: D23.2 (A), MX23.2 (ROW)
- new net: D24.2 (A), MX24.2 (ROW)
- new net: D25.2 (A), MX25.2 (ROW)
- new net: D26.2 (A), MX26.2 (ROW)
- new net: D27.2 (A), MX27.2 (ROW)
- new net: D28.2 (A), MX28.2 (ROW)
- new net: D29.2 (A), MX29.2 (ROW)
- new net: D30.2 (A), MX30.2 (ROW)
- new net: D31.2 (A), MX31.2 (ROW), MX32.2 (ROW)
- new net: D37.2 (A), MX38.2 (ROW)
- new net: D38.2 (A), MX39.2 (ROW)
- new net: D39.2 (A), MX40.2 (ROW)
- new net: D40.2 (A), MX41.2 (ROW)
- new net: D41.2 (A), MX42.2 (ROW)
- new net: D42.2 (A), MX43.2 (ROW)
- new net: D43.2 (A), MX44.2 (ROW)
- new net: D44.2 (A), MX45.2 (ROW)
- new net: D45.2 (A), MX46.2 (ROW)
- new net: D46.2 (A), MX47.2 (ROW)
- new net: D47.2 (A), MX48.2 (ROW)
- new net: D48.2 (A), MX49.2 (ROW)
- new net: D54.2 (A), MX56.2 (ROW)
- new net: D55.2 (A), MX57.2 (ROW)
- new net: D56.2 (A), MX58.2 (ROW)
- new net: D57.2 (A), MX59.2 (ROW)
- new net: D58.2 (A), MX60.2 (ROW)
- new net: D59.2 (A), MX61.2 (ROW)
- new net: D60.2 (A), MX62.2 (ROW)
- new net: D61.2 (A), MX63.2 (ROW)
- new net: D62.2 (A), MX64.2 (ROW)
- new net: D63.2 (A), MX65.2 (ROW)
- new net: D64.2 (A), MX66.2 (ROW)
- new net: D67.2 (A), MX69.2 (ROW)
- new net: D68.2 (A), MX70.2 (ROW)
- new net: D69.2 (A), MX71.2 (ROW)
- new net: D70.2 (A), MX72.2 (ROW)
- new net: D71.2 (A), MX73.2 (ROW)
- new net: D72.2 (A), MX74.2 (ROW)
- new net: D73.2 (A), MX75.2 (ROW)
- new net: D74.2 (A), MX76.2 (ROW)
- new net: D83.2 (A), MX86.2 (ROW)
- new net: D80.2 (A), MX83.2 (ROW)
- new net: D81.2 (A), MX84.2 (ROW)
- new net: D82.2 (A), MX85.2 (ROW)
- new net: D66.2 (A), MX68.2 (ROW)
- new net: D53.2 (A), MX54.2 (ROW), MX55.2 (ROW)
- new net: D36.2 (A), MX37.2 (ROW)
- new net: D49.2 (A), MX50.2 (ROW)
- new net: D65.2 (A), MX67.2 (ROW)
- new net: D77.2 (A), MX79.2 (ROW), MX80.2 (ROW)
- new net: D85.2 (A), MX88.2 (ROW)
- new net: D84.2 (A), MX87.2 (ROW)
- new net: D86.2 (A), MX89.2 (ROW)
- new net: D2.2 (A), MX2.2 (ROW)
- new net: D3.2 (A), MX3.2 (ROW)
- new net: D4.2 (A), MX4.2 (ROW)
- new net: D5.2 (A), MX5.2 (ROW)
- new net: D6.2 (A), MX6.2 (ROW)
- new net: D7.2 (A), MX7.2 (ROW)
- new net: D8.2 (A), MX8.2 (ROW)
- new net: D9.2 (A), MX9.2 (ROW)
- new net: D10.2 (A), MX10.2 (ROW)
- new net: D11.2 (A), MX11.2 (ROW)
- new net: D12.2 (A), MX12.2 (ROW)
- new net: D13.2 (A), MX13.2 (ROW)
- new net: D33.2 (A), MX34.2 (ROW)
- new net: D34.2 (A), MX35.2 (ROW)
- new net: D35.2 (A), MX36.2 (ROW)
- new net: D50.2 (A), MX51.2 (ROW)
- new net: D51.2 (A), MX52.2 (ROW)
- new net: D52.2 (A), MX53.2 (ROW)
- new net: MX54.3 (LED), MX55.3 (LED), R4.1
- new net: D32.2 (A), MX33.2 (ROW)
- new net: D78.2 (A), MX81.2 (ROW)
- new net CAPS_LED: R4.2
- new net Col0: MX1.1 (COL), MX18.1 (COL), MX37.1 (COL), MX54.1 (COL), MX55.1 (COL), MX68.1 (COL), MX83.1 (COL)
- new net Col1: MX19.1 (COL), MX2.1 (COL), MX38.1 (COL), MX56.1 (COL), MX69.1 (COL), MX84.1 (COL)
- new net Col10: MX11.1 (COL), MX28.1 (COL), MX47.1 (COL), MX65.1 (COL), MX78.1 (COL), MX87.1 (COL)
- new net Col11: MX12.1 (COL), MX29.1 (COL), MX48.1 (COL), MX66.1 (COL), MX88.1 (COL)
- new net Col12: MX13.1 (COL), MX30.1 (COL), MX49.1 (COL), MX67.1 (COL), MX79.1 (COL), MX80.1 (COL)
- new net Col13: MX14.1 (COL), MX31.1 (COL), MX32.1 (COL), MX33.1 (COL), MX50.1 (COL), MX81.1 (COL), MX89.1 (COL)
- new net Col14: MX15.1 (COL), MX34.1 (COL), MX51.1 (COL), MX90.1 (COL)
- new net Col15: MX16.1 (COL), MX35.1 (COL), MX52.1 (COL), MX82.1 (COL), MX91.1 (COL)
- new net Col16: MX17.1 (COL), MX36.1 (COL), MX53.1 (COL), MX92.1 (COL)
- new net Col2: MX20.1 (COL), MX3.1 (COL), MX39.1 (COL), MX57.1 (COL), MX70.1 (COL), MX85.1 (COL)
- new net Col3: MX21.1 (COL), MX4.1 (COL), MX40.1 (COL), MX58.1 (COL), MX71.1 (COL)
- new net Col4: MX22.1 (COL), MX41.1 (COL), MX5.1 (COL), MX59.1 (COL), MX72.1 (COL)
- new net Col5: MX23.1 (COL), MX42.1 (COL), MX6.1 (COL), MX60.1 (COL), MX73.1 (COL)
- new net Col6: MX24.1 (COL), MX43.1 (COL), MX61.1 (COL), MX7.1 (COL), MX74.1 (COL), MX86.1 (COL)
- new net Col7: MX25.1 (COL), MX44.1 (COL), MX62.1 (COL), MX75.1 (COL), MX8.1 (COL)
- new net Col8: MX26.1 (COL), MX45.1 (COL), MX63.1 (COL), MX76.1 (COL), MX9.1 (COL)
- new net Col9: MX10.1 (COL), MX27.1 (COL), MX46.1 (COL), MX64.1 (COL), MX77.1 (COL)
- new net Row0: D1.1 (K), D10.1 (K), D11.1 (K), D12.1 (K), D13.1 (K), D14.1 (K), D15.1 (K), D16.1 (K), D17.1 (K), D2.1 (K), D3.1 (K), D4.1 (K), D5.1 (K), D6.1 (K), D7.1 (K), D8.1 (K), D9.1 (K)
- new net Row1: D18.1 (K), D19.1 (K), D20.1 (K), D21.1 (K), D22.1 (K), D23.1 (K), D24.1 (K), D25.1 (K), D26.1 (K), D27.1 (K), D28.1 (K), D29.1 (K), D30.1 (K), D31.1 (K), D33.1 (K), D34.1 (K), D35.1 (K)
- new net Row2: D36.1 (K), D37.1 (K), D38.1 (K), D39.1 (K), D40.1 (K), D41.1 (K), D42.1 (K), D43.1 (K), D44.1 (K), D45.1 (K), D46.1 (K), D47.1 (K), D48.1 (K), D49.1 (K), D50.1 (K), D51.1 (K), D52.1 (K)
- new net Row3: D32.1 (K), D53.1 (K), D54.1 (K), D55.1 (K), D56.1 (K), D57.1 (K), D58.1 (K), D59.1 (K), D60.1 (K), D61.1 (K), D62.1 (K), D63.1 (K), D64.1 (K), D65.1 (K)
- new net Row4: D66.1 (K), D67.1 (K), D68.1 (K), D69.1 (K), D70.1 (K), D71.1 (K), D72.1 (K), D73.1 (K), D74.1 (K), D75.1 (K), D76.1 (K), D77.1 (K), D78.1 (K), D79.1 (K)
- new net Row5: D80.1 (K), D81.1 (K), D82.1 (K), D83.1 (K), D84.1 (K), D85.1 (K), D86.1 (K), D87.1 (K), D88.1 (K), D89.1 (K)
Other:
- moved on the sheet: C1, C10, C11, C12, C2, C3, C4, C5, C6, C7, C8, C9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

Commit message: preliminary component placement, update submodule
Parts:
- MX79: footprint MX_Only:MXOnly-1U-NoLED -> MX_Only:MXOnly-1.75U-NoLED
Connections:
- net CAPS_LED: now also R4.1; no longer R4.2
- net GND: now also MX54.3 (LED), MX55.3 (LED); no longer MX54.4 (LEDGND), MX55.4 (LEDGND)
- new net: MX54.4 (LEDGND), MX55.4 (LEDGND), R4.2
Other:
- moved on the sheet: R4
Changed lines of the file:
@@
 L Device:R_Small R4
 U 1 1 60CB7107
-P 3100 11050
-F 0 "R4" H 3200 11050 50  0000 C CNN
-F 1 "1k" H 3200 11150 50  0000 C CNN
-F 2 "Resistor_SMD:R_0603_1608Metric" H 3100 11050 50  0001 C CNN
-F 3 "~" H 3100 11050 50  0001 C CNN
-	1    3100 11050
-	-1   0    0    1
+P 3000 11250
+F 0 "R4" H 3100 11250 50  0000 C CNN
+F 1 "1k" H 3100 11350 50  0000 C CNN
+F 2 "Resistor_SMD:R_0603_1608Metric" H 3000 11250 50  0001 C CNN
+F 3 "~" H 3000 11250 50  0001 C CNN
+	1    3000 11250
+	0    -1   -1   0
 $EndComp
 $Comp
 L power:GND #PWR016
 U 1 1 60CBB4C0
-P 2950 11250
-F 0 "#PWR016" H 2950 11000 50  0001 C CNN
-F 1 "GND" H 2955 11077 50  0000 C CNN
-F 2 "" H 2950 11250 50  0001 C CNN
-F 3 "" H 2950 11250 50  0001 C CNN
-	1    2950 11250
+P 3000 10850
+F 0 "#PWR016" H 3000 10600 50  0001 C CNN
+F 1 "GND" H 3005 10677 50  0000 C CNN
+F 2 "" H 3000 10850 50  0001 C CNN
+F 3 "" H 3000 10850 50  0001 C CNN
+	1    3000 10850
 	1    0    0    -1
 $EndComp
@@
 	1    0    0    -1
 $EndComp
-Text GLabel 3100 10900 0    50   Input ~ 0
+Text GLabel 2800 11250 1    50   Input ~ 0
 CAPS_LED
 Wire Wire Line
@@
 Wire Wire Line
 	2000 11500 3550 11500
-Connection ~ 3250 11250
 Wire Wire Line
 	3350 11150 3100 11150
 Connection ~ 3350 11150
-Wire Wire Line
-	3100 10950 3100 10900
-Wire Wire Line
-	2950 11250 3250 11250
 $Comp
 L MX_Alps_Hybrid:MX-NoLED MX31
@@
 F 0 "MX79" H 15533 12373 60  0000 C CNN
 F 1 "MX-NoLED" H 15533 12299 20  0000 C CNN
-F 2 "MX_Only:MXOnly-1U-NoLED" H 14875 12125 60  0001 C CNN
+F 2 "MX_Only:MXOnly-1.75U-NoLED" H 14875 12125 60  0001 C CNN
 F 3 "" H 14875 12125 60  0001 C CNN
 	1    15500 12150
@@
 Wire Wire Line
 	10050 13500 5900 13500
+Wire Wire Line
+	2800 11250 2900 11250
+Wire Wire Line
+	3100 11250 3250 11250
+Connection ~ 3250 11250
+Wire Wire Line
+	3100 11150 3100 10850
+Wire Wire Line
+	3100 10850 3000 10850
 $EndSCHEMATC

Commit message: lots of changes
Parts:
- removed MX16: MX-NoLED, MX_Only:MXOnly-1U-NoLED, symbol MX_Alps_Hybrid:MX-NoLED
- added D90: D_Schottky, Diode_SMD:D_SOD-123, symbol Device:D_Schottky
- added D91: D_TVS, Diode_SMD:D_SOD-123, symbol Device:D_TVS
- added F1: 500mA, Fuse:Fuse_1206_3216Metric, symbol Device:Polyfuse_Small
- added LOGO1, LOGO2: O-LOGO, board_logos:o-logo-300dpi, symbol logos:O-LOGO
- added MX16: MX-LED, MX_Only:MXOnly-1U, symbol MX_Alps_Hybrid:MX-LED
- added R5: 1k, Resistor_SMD:R_0603_1608Metric, symbol Device:R_Small
Connections:
- net CAPS_LED is gone; now on net CAPS: R4.1
- net +3V3: now also D90.2 (A)
- net +5V: now also MX54.3 (LED), MX55.3 (LED), D90.1 (K), D91.2 (A2), F1.1, MX16.3 (LED); no longer J1.1 (Pin_1)
- net Col0: now also MX54.2 (ROW), U2.31 (PA10); no longer MX54.1 (COL)
- net Col1: now also U2.30 (PA9)
- net Col10: now also U2.19 (PB1)
- net Col11: now also U2.18 (PB0)
- net Col12: now also U2.17 (PA7)
- net Col13: now also U2.12 (PA2)
- net Col14: now also U2.45 (PB8)
- net Col15: now also U2.42 (PB6), MX16.1 (COL)
- net Col16: now also U2.41 (PB5)
- net Col2: now also U2.29 (PA8)
- net Col3: now also U2.28 (PB15)
- net Col4: now also U2.27 (PB14)
- net Col5: now also U2.26 (PB13)
- net Col6: now also U2.25 (PB12)
- net Col7: now also U2.22 (PB11)
- net Col8: now also U2.21 (PB10)
- net Col9: now also U2.20 (PB2)
- net GND: now also D91.1 (A1); no longer MX54.3 (LED), MX55.3 (LED)
- net Row0: now also U2.16 (PA6)
- net Row1: now also U2.39 (PB3)
- net Row2: now also U2.40 (PB4)
- net Row3: now also U2.15 (PA5)
- net Row4: now also U2.13 (PA3)
- net Row5: now also U2.14 (PA4)
- net SCROLL: now reaches U2.38 (PA15)
- net SCROLL: now also R5.2
- net CAPS: now reaches U2.43 (PB7)
- net at D16.2 (A): now also MX16.2 (ROW)
- net at MX77.2 (ROW): now also D75.2 (A)
- net at MX78.2 (ROW): now also D76.2 (A)
- net at D53.2 (A), MX55.2 (ROW): now also MX54.1 (COL); no longer MX54.2 (ROW)
- new net: MX16.4 (LEDGND), R5.1
- new net VCC: F1.2, J1.1 (Pin_1)
Other:
- moved on the sheet: C1, C2, U1
